File: RecoveryBoard/eagle/RecoveryBoard.brd (EAGLE design)
At the start: 120.9 x 54.6 mm, 96 parts, among them Q1 BSS123, Q2 BSS123, Q3 BSS123, Q4 BPR-301, Q5 BPR-301, Q6 MOSFET-PCH-SOT23-6, U1 STM32F042K6, U10 TPS63070, U2 BD62120AEFJ-E2, U3 H11F1SR2M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

Commit message: added camera board folder and git ignore
Parts:
- R26, R27: value 51.1 -> 51
Changed lines of the file:
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@@
 <attribute name="VALUE" x="62.3" y="22.75" size="0.4064" layer="27" font="vector" ratio="15"/>
 </element>
-<element name="R26" library="oresat-rcl" package=".0603-C-NOSILK" value="51.1" x="28" y="15.5" smashed="yes" rot="R270">
+<element name="R26" library="oresat-rcl" package=".0603-C-NOSILK" value="51" x="28" y="15.5" smashed="yes" rot="R270">
 <attribute name="NAME" x="28.365" y="12.625" size="0.635" layer="25" font="vector" ratio="20" rot="R90"/>
 <attribute name="VALUE" x="26.095" y="16.135" size="0.4064" layer="27" rot="R270"/>
 </element>
-<element name="R27" library="oresat-rcl" package=".0603-C-NOSILK" value="51.1" x="28" y="6" smashed="yes" rot="R270">
+<element name="R27" library="oresat-rcl" package=".0603-C-NOSILK" value="51" x="28" y="6" smashed="yes" rot="R270">
 <attribute name="NAME" x="28.305" y="3.125" size="0.635" layer="25" font="vector" ratio="20" rot="R90"/>
 <attribute name="VALUE" x="26.095" y="6.635" size="0.4064" layer="27" rot="R270"/>

Commit message: file names
Parts:
- R8, R9: value 442 -> 470
Changed lines of the file:
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@@
 <attribute name="VALUE" x="13.005" y="47.465" size="0.4064" layer="27" rot="R90"/>
 </element>
-<element name="R8" library="oresat-rcl" package=".0603-C-NOSILK" value="442" x="15.1" y="41.3" smashed="yes" rot="R90">
+<element name="R8" library="oresat-rcl" package=".0603-C-NOSILK" value="470" x="15.1" y="41.3" smashed="yes" rot="R90">
 <attribute name="NAME" x="16.365" y="40.865" size="0.635" layer="25" font="vector" ratio="20" rot="R90"/>
 <attribute name="VALUE" x="17.005" y="40.665" size="0.4064" layer="27" rot="R90"/>
 </element>
-<element name="R9" library="oresat-rcl" package=".0603-C-NOSILK" value="442" x="104.77" y="48.39" smashed="yes" rot="R180">
+<element name="R9" library="oresat-rcl" package=".0603-C-NOSILK" value="470" x="104.77" y="48.39" smashed="yes" rot="R180">
 <attribute name="NAME" x="104.195" y="47.045" size="0.635" layer="25" font="vector" ratio="20"/>
 <attribute name="VALUE" x="105.405" y="50.295" size="0.4064" layer="27" rot="R180"/>
