File: controlSystem/RecoveryBoard/eagle/RecoveryBoard.sch (EAGLE design)
At the start: 104 parts, among them Q1 BSS123, Q2 BSS123, Q3 BSS123, Q4 BPR-301, Q5 BPR-301, Q6 MOSFET-PCH-SOT23-6, Q7 SI7465DP-T1-E3, U1 STM32F042K6, U10 TPS63070, U2 BD62120AEFJ-E2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

Commit message: added fastener restrictions and more satisfying via placement
Other:
- note added: "12V Out at 1A"
Changed lines of the file:
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@@
 <wire x1="73.66" y1="167.64" x2="74.93" y2="167.64" width="0.1524" layer="97"/>
 <text x="60.325" y="136.525" size="1.778" layer="97">USART Connector for Laptop</text>
+<text x="239.395" y="191.135" size="1.778" layer="97">12V Out at 1A</text>
 </plain>
 <instances>
