File: controlSystem/RecoveryBoard/eagle/RecoveryBoard.sch (EAGLE design)
At the start: 104 parts, among them Q1 BSS123, Q2 BSS123, Q3 BSS123, Q4 BPR-301, Q5 BPR-301, Q6 MOSFET-PCH-SOT23-6, Q7 SI7465DP-T1-E3, U1 STM32F042K6, U10 TPS63070, U2 BD62120AEFJ-E2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

Commit message: First big checkpoint of recovery-firmware: STM32 is using HSE crystal, serial port, and tools seem to be working correctly. Committing new schematic and board file with updated names, but no electrical or layout changes.
Connections:
- net ACOK renamed UMB_ON
- net DCMDIR renamed DCM_DIR
- net DCM_ON renamed DCM_PWR
- net ISO-CHUTE renamed ISO_MAIN
- net ISO-DROGUE renamed ISO_DROGUE
- net LA_IN1 renamed LA_DRV1
- net LA_IN2 renamed LA_DRV2
- net SENSOR1 renamed ROTSENE1
- net SENSOR2 renamed ROTSENSE2
- net SENSOR_ON renamed ROTSENSE_PWR
Other:
- note added: "(~0.3, ~ 1, ~ 2) A"
- note added: "16 MHz"
- note added: "DCM_SPEED floats up to 5V?!"
- note added: "NEEDS 1K RESISTOR OR SOMETHING"
- note added: "PWM (BLU)"
- note added: "PWM = 0% DC = Motor off"
- note added: "Rotation Sensor"
- note removed: "Light Sensor"
- note removed: "PWM OUT (BLU)"
- note removed: "Use the pull up resistor in the STM with this...there is a resistor in the motor"
- moved on the sheet: C3, C4, D5, Q2, Q4, Q5, R10, R31, R36, R7, R8, R9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

Commit message: Spun off blinky to a separate file, added shell commands, added polling for telemetrum signals, and updated board file with better names for signals (no changes to layout or schematic).
Connections:
- net CHUTE renamed T_MAIN
- net DROGUE renamed T_DROGUE
- net T_GND renamed T_VLIPO
Changed lines of the file:
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@@
 <setting verticaltext="up"/>
 </settings>
-<grid distance="0.05" unitdist="inch" unit="inch" style="lines" multiple="2" display="no" altdistance="0.01" altunitdist="inch" altunit="inch"/>
+<grid distance="0.1" unitdist="inch" unit="inch" style="lines" multiple="1" display="no" altdistance="0.01" altunitdist="inch" altunit="inch"/>
 <layers>
 <layer number="1" name="Top" color="4" fill="1" visible="no" active="no"/>
@@
 </segment>
 </net>
-<net name="CHUTE" class="0">
+<net name="T_MAIN" class="0">
 <segment>
 <label x="102.87" y="175.26" size="1.778" layer="95" xref="yes"/>
@@
 </segment>
 </net>
-<net name="DROGUE" class="0">
+<net name="T_DROGUE" class="0">
 <segment>
 <label x="102.87" y="171.45" size="1.778" layer="95" xref="yes"/>
@@
 </segment>
 </net>
-<net name="T_GND" class="0">
+<net name="T_VLIPO" class="0">
 <segment>
 <label x="102.87" y="167.64" size="1.778" layer="95" xref="yes"/>
@@
 </segment>
 </net>
-<net name="T_GND" class="0">
+<net name="T_VLIPO" class="0">
 <segment>
 <wire x1="185.42" y1="287.02" x2="198.12" y2="287.02" width="0.1524" layer="91"/>
@@
 </segment>
 </net>
-<net name="CHUTE" class="0">
+<net name="T_MAIN" class="0">
 <segment>
 <wire x1="198.12" y1="341.63" x2="198.12" y2="342.9" width="0.1524" layer="91"/>
@@
 </segment>
 </net>
-<net name="DROGUE" class="0">
+<net name="T_DROGUE" class="0">
 <segment>
 <wire x1="250.19" y1="341.63" x2="250.19" y2="355.6" width="0.1524" layer="91"/>

Commit message: Moved libraries to sub folder, added some comments in the schematic.
Other:
- note added: "M+ (RED)"
- note added: "M- (BLK)"
- note added: "POT (PUR)"
- note added: "POT+ (YLW)"
- note added: "POT- (ORG)"
- note added: "SHORT TO POWER DOWN"
- note removed: "SHORT TO DISARM"
- moved on the sheet: J2
Changed lines of the file:
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@@
 <text x="72.39" y="190.5" size="1.778" layer="95">Outside World</text>
 <text x="327.66" y="176.53" size="1.778" layer="97">TO 3S1P battery</text>
-<text x="49.53" y="180.34" size="1.778" layer="97">SHORT TO DISARM</text>
+<text x="41.91" y="180.34" size="1.778" layer="97">SHORT TO POWER DOWN</text>
 <text x="57.15" y="175.26" size="1.778" layer="97">19V umbilical</text>
 <text x="308.61" y="231.14" size="1.778" layer="97">12V power switch</text>
@@
 <text x="453.39" y="271.78" size="1.778" layer="97">DCM_SPEED floats up to 5V?!</text>
 <text x="453.39" y="267.97" size="1.778" layer="97">PWM = 0% DC = Motor off</text>
+<text x="431.8" y="215.9" size="1.778" layer="97">POT- (ORG)</text>
+<text x="431.8" y="213.36" size="1.778" layer="97">POT  (PUR)</text>
+<text x="431.8" y="210.82" size="1.778" layer="97">M+   (RED)</text>
+<text x="431.8" y="208.28" size="1.778" layer="97">M-   (BLK)</text>
+<text x="431.8" y="205.74" size="1.778" layer="97">POT+ (YLW)</text>
 </plain>
 <instances>
@@
 <attribute name="DRAWING_NAME" x="469.9" y="19.05" size="2.54" layer="94"/>
 </instance>
-<instance part="J2" gate="A" x="458.47" y="210.82" smashed="yes" rot="MR0">
-<attribute name="NAME" x="464.82" y="219.075" size="1.778" layer="95" rot="MR0"/>
-<attribute name="VALUE" x="464.82" y="200.66" size="1.778" layer="96" rot="MR0"/>
+<instance part="J2" gate="A" x="448.31" y="210.82" smashed="yes" rot="MR0">
+<attribute name="NAME" x="454.66" y="219.075" size="1.778" layer="95" rot="MR0"/>
+<attribute name="VALUE" x="454.66" y="200.66" size="1.778" layer="96" rot="MR0"/>
 </instance>
 <instance part="J1" gate="A" x="471.17" y="292.1" smashed="yes">
@@
 <segment>
 <pinref part="J2" gate="A" pin="1"/>
-<wire x1="461.01" y1="215.9" x2="488.95" y2="215.9" width="0.1524" layer="91"/>
+<wire x1="450.85" y1="215.9" x2="488.95" y2="215.9" width="0.1524" layer="91"/>
 <pinref part="SUPPLY40" gate="GND" pin="GND"/>
 <wire x1="488.95" y1="215.9" x2="488.95" y2="199.39" width="0.1524" layer="91"/>
-<label x="464.82" y="215.9" size="1.778" layer="95"/>
+<label x="457.2" y="215.9" size="1.778" layer="95"/>
 </segment>
 </net>
@@
 <segment>
 <pinref part="J2" gate="A" pin="5"/>
-<wire x1="461.01" y1="205.74" x2="485.14" y2="205.74" width="0.1524" layer="91"/>
-<label x="464.82" y="205.74" size="1.778" layer="95"/>
+<wire x1="450.85" y1="205.74" x2="485.14" y2="205.74" width="0.1524" layer="91"/>
+<label x="457.2" y="205.74" size="1.778" layer="95"/>
 <pinref part="SUPPLY41" gate="G$1" pin="3.3V"/>
 <wire x1="485.14" y1="205.74" x2="485.14" y2="223.52" width="0.1524" layer="91"/>
@@
 <pinref part="U2" gate="G$1" pin="OUT1"/>
 <pinref part="J2" gate="A" pin="3"/>
-<wire x1="497.84" y1="210.82" x2="461.01" y2="210.82" width="0.1524" layer="91"/>
-<label x="464.82" y="210.82" size="1.778" layer="95"/>
+<wire x1="497.84" y1="210.82" x2="450.85" y2="210.82" width="0.1524" layer="91"/>
+<label x="457.2" y="210.82" size="1.778" layer="95"/>
 </segment>
 </net>
@@
 <label x="299.72" y="203.2" size="1.27" layer="95"/>
 <pinref part="J2" gate="A" pin="2"/>
-<wire x1="461.01" y1="213.36" x2="480.06" y2="213.36" width="0.1524" layer="91"/>
+<wire x1="450.85" y1="213.36" x2="480.06" y2="213.36" width="0.1524" layer="91"/>
 <wire x1="480.06" y1="180.34" x2="480.06" y2="213.36" width="0.1524" layer="91"/>
-<label x="464.82" y="213.36" size="1.778" layer="95"/>
+<label x="457.2" y="213.36" size="1.778" layer="95"/>
 <wire x1="480.06" y1="180.34" x2="401.32" y2="180.34" width="0.1524" layer="91"/>
 <wire x1="401.32" y1="180.34" x2="358.14" y2="180.34" width="0.1524" layer="91"/>
@@
 <segment>
 <pinref part="J2" gate="A" pin="4"/>
-<label x="464.82" y="208.28" size="1.778" layer="95"/>
-<wire x1="461.01" y1="208.28" x2="500.38" y2="208.28" width="0.1524" layer="91"/>
+<label x="457.2" y="208.28" size="1.778" layer="95"/>
+<wire x1="450.85" y1="208.28" x2="500.38" y2="208.28" width="0.1524" layer="91"/>
 <pinref part="U2" gate="G$1" pin="OUT2"/>
 <wire x1="500.38" y1="208.28" x2="500.38" y2="156.21" width="0.1524" layer="91"/>
