File: controlSystem/RecoveryBoard/eagle/RecoveryBoard.brd (EAGLE design)
At the start: 120.9 x 54.6 mm, 104 parts, among them Q1 BSS123, Q2 BSS123, Q3 BSS123, Q4 BPR-301, Q5 BPR-301, Q6 MOSFET-PCH-SOT23-6, Q7 SI7465DP-T1-E3, U1 STM32F042K6, U10 TPS63070, U2 BD62120AEFJ-E2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

Commit message: First big checkpoint of recovery-firmware: STM32 is using HSE crystal, serial port, and tools seem to be working correctly. Committing new schematic and board file with updated names, but no electrical or layout changes.
Connections:
- net ACOK renamed UMB_ON
- net DCMDIR renamed DCM_DIR
- net DCM_ON renamed DCM_PWR
- net ISO-CHUTE renamed ISO_MAIN
- net ISO-DROGUE renamed ISO_DROGUE
- net LA_IN1 renamed LA_DRV1
- net LA_IN2 renamed LA_DRV2
- net SENSOR1 renamed ROTSENE1
- net SENSOR2 renamed ROTSENSE2
- net SENSOR_ON renamed ROTSENSE_PWR
Changed lines of the file:
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@@
 <?xml version="1.0" encoding="utf-8"?>
 <!DOCTYPE eagle SYSTEM "eagle.dtd">
-<eagle version="9.6.1">
+<eagle version="9.6.2">
 <drawing>
 <settings>
@@
 <wire x1="56.4" y1="37.82" x2="56.4" y2="37.1" width="0.35" layer="1"/>
 </signal>
-<signal name="ACOK">
+<signal name="UMB_ON">
 <contactref element="U$5" pad="!ACOK"/>
 <contactref element="R19" pad="1"/>
@@
 <wire x1="62.5" y1="5.5" x2="62.5" y2="8" width="0.2" layer="1"/>
 </signal>
-<signal name="LA_IN1">
+<signal name="LA_DRV1">
 <contactref element="U1" pad="18"/>
 <contactref element="R32" pad="1"/>
@@
 <wire x1="85.5" y1="2" x2="85.5" y2="3.993" width="0.2" layer="1"/>
 </signal>
-<signal name="LA_IN2">
+<signal name="LA_DRV2">
 <contactref element="U1" pad="19"/>
 <contactref element="R33" pad="1"/>
@@
 <wire x1="86.8" y1="2" x2="86.8" y2="4.023" width="0.2" layer="1"/>
 </signal>
-<signal name="SENSOR1">
+<signal name="ROTSENE1">
 <contactref element="R7" pad="2"/>
 <contactref element="U1" pad="28"/>
@@
 <wire x1="85.1" y1="37.8" x2="90.4" y2="37.8" width="0.2" layer="16"/>
 </signal>
-<signal name="DCMDIR">
+<signal name="DCM_DIR">
 <contactref element="J1" pad="3"/>
 <contactref element="R12" pad="1"/>
@@
 <wire x1="89.8" y1="22.8" x2="77.3" y2="10.3" width="0.2" layer="16"/>
 </signal>
-<signal name="SENSOR_ON">
+<signal name="ROTSENSE_PWR">
 <contactref element="R36" pad="1"/>
 <contactref element="U1" pad="26"/>
@@
 <wire x1="97.58" y1="38.48" x2="97.7" y2="38.6" width="0.2" layer="1"/>
 </signal>
-<signal name="SENSOR2">
+<signal name="ROTSENSE2">
 <contactref element="R10" pad="2"/>
 <contactref element="U1" pad="27"/>
@@
 <wire x1="81.3" y1="11.2" x2="80.6" y2="11.9" width="0.2" layer="1"/>
 </signal>
-<signal name="DCM_ON">
+<signal name="DCM_PWR">
 <contactref element="R35" pad="1"/>
 <contactref element="U1" pad="13"/>
@@
 <wire x1="30.66" y1="6.7" x2="30.9" y2="6.46" width="0.5" layer="1"/>
 </signal>
-<signal name="ISO-CHUTE">
+<signal name="ISO_MAIN">
 <contactref element="R28" pad="1"/>
 <contactref element="U3" pad="OUT"/>
@@
 <wire x1="49.3" y1="14.9" x2="60.2" y2="14.9" width="0.3" layer="16"/>
 </signal>
-<signal name="ISO-DROGUE">
+<signal name="ISO_DROGUE">
 <contactref element="R29" pad="1"/>
 <contactref element="U5" pad="OUT"/>

Commit message: Spun off blinky to a separate file, added shell commands, added polling for telemetrum signals, and updated board file with better names for signals (no changes to layout or schematic).
Connections:
- net CHUTE renamed T_MAIN
- net DROGUE renamed T_DROGUE
- net T_GND renamed T_VLIPO
Changed lines of the file:
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@@
 <wire x1="55.595" y1="17.795" x2="55.595" y2="15.155" width="1" layer="1"/>
 </signal>
-<signal name="CHUTE">
+<signal name="T_MAIN">
 <contactref element="U3" pad="ANOD"/>
 <contactref element="JP2" pad="5"/>
@@
 <wire x1="27.85" y1="18.7" x2="30.9" y2="18.7" width="0.5" layer="1"/>
 </signal>
-<signal name="DROGUE">
+<signal name="T_DROGUE">
 <contactref element="U5" pad="ANOD"/>
 <contactref element="JP2" pad="6"/>
@@
 <wire x1="27.85" y1="9" x2="30.9" y2="9" width="0.5" layer="1"/>
 </signal>
-<signal name="T_GND">
+<signal name="T_VLIPO">
 <contactref element="R26" pad="2"/>
 <contactref element="R27" pad="2"/>
