File: controlSystem/SpringPinBoards/ActiveModule/ActiveModule.kicad_pcb (KiCad board)
At the start: 2 copper layers, 18.7 x 13.3 mm, 9 parts, among them J1 Conn_01x01_Male, J2 Conn_01x01_Male, J3 Conn_01x01_Male, J4 Conn_01x01_Male, J5 Conn_01x01_Male, J6 Conn_01x01_Male, J7 Conn_01x06

Commit message: Design review changes
Other:
- board text added: "2022/09/19"
- board text added: "Active Module Spring Pin Board"
- board text added: "PSAS ERS"
- board text removed: "2022/09/19 PSAS ERS Active Module Spring Pin Board"
Changed lines of the file:
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@@
     (pad "" np_thru_hole circle (at 0 0) (size 2.2 2.2) (drill 2.2) (layers *.Cu *.Mask))
   )
+  (gr_circle (center 154.494375 78.657) (end 156.875625 78.657) (layer "F.Mask") (width 0.2) (fill solid))
+  (gr_circle (center 144.175625 78.657) (end 146.556875 78.657) (layer "F.Mask") (width 0.2) (fill solid))
   (gr_arc (start 157.11375 69.132) (mid 158.236282 69.596968) (end 158.70125 70.7195) (layer "Dwgs.User") (width 0.2))
   (gr_line (start 141.55625 69.132) (end 157.11375 69.132) (layer "Dwgs.User") (width 0.2))
@@
   (gr_arc (start 141.55625 82.467) (mid 140.433718 82.002032) (end 139.96875 80.8795) (layer "Edge.Cuts") (width 0.2))
   (gr_line (start 139.96875 80.8795) (end 139.96875 70.7195) (layer "Edge.Cuts") (width 0.2))
-  (gr_text "2022/09/19 PSAS ERS\nActive Module Spring Pin Board" (at 140.9 81.1) (layer "F.SilkS")
-    (effects (font (size 0.5 0.5) (thickness 0.12)) (justify left))
+  (gr_text "2022/09/19\n\n" (at 149.3 79.9) (layer "F.SilkS")
+    (effects (font (size 0.5 0.5) (thickness 0.12)))
+  )
+  (gr_text "Active Module Spring Pin Board" (at 149.3 81.6) (layer "F.SilkS")
+    (effects (font (size 0.5 0.5) (thickness 0.12)))
+  )
+  (gr_text "PSAS ERS" (at 149.3 80.6) (layer "F.SilkS")
+    (effects (font (size 0.5 0.5) (thickness 0.12)))
   )
   (segment (start 141.25 71.35) (end 141.8 70.8) (width 1) (layer "F.Cu") (net 1))
