File: controlSystem/SpringPinBoards/PassiveModule/PassiveModule.kicad_pcb (KiCad board)
At the start: 2 copper layers, 17.9 x 13.3 mm, 9 parts, among them J1 Conn_01x01_Male, J2 Conn_01x01_Male, J3 Conn_01x01_Male, J4 Conn_01x01_Male, J5 Conn_01x01_Male, J6 Conn_01x01_Male, J7 Conn_02x03_Odd_Even

Commit message: Design review changes
Other:
- board text added: "2022/09/19"
- board text added: "PSAS ERS"
- board text added: "Passive Module Spring Pin Board"
- board text removed: "2022/09/19 PSAS ERS Passive Module Spring Pin Board"
Changed lines of the file:
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@@
     )
   )
-  (gr_circle locked (center 174.275478 89.0575) (end 176.358278 89.0575) (layer "Dwgs.User") (width 0.2) (fill none))
+  (gr_circle (center 174.275478 89.0575) (end 176.358278 89.0575) (layer "B.Mask") (width 0.2) (fill solid))
+  (gr_circle (center 179.362966 89.0575) (end 181.445766 89.0575) (layer "B.Mask") (width 0.2) (fill solid))
   (gr_arc locked (start 186.343897 79.5325) (mid 187.711707 80.314238) (end 187.732406 81.889545) (layer "Dwgs.User") (width 0.2))
   (gr_line locked (start 175.370897 86.581147) (end 173.243603 86.581147) (layer "Dwgs.User") (width 0.2))
@@
   (gr_arc locked (start 175.370897 82.9615) (mid 176.493429 83.426468) (end 176.958397 84.549) (layer "Dwgs.User") (width 0.2))
   (gr_arc locked (start 173.243603 86.581147) (mid 172.121071 86.116179) (end 171.656103 84.993647) (layer "Dwgs.User") (width 0.2))
+  (gr_circle locked (center 174.275478 89.0575) (end 176.358278 89.0575) (layer "Dwgs.User") (width 0.2) (fill none))
   (gr_line locked (start 171.656103 84.993647) (end 171.656103 84.549) (layer "Dwgs.User") (width 0.2))
   (gr_arc locked (start 171.656103 92.8675) (mid 170.533571 92.402532) (end 170.068603 91.28) (layer "Dwgs.User") (width 0.2))
   (gr_line locked (start 170.068603 81.12) (end 170.068603 91.28) (layer "Dwgs.User") (width 0.2))
   (gr_circle locked (center 179.434853 84.2315) (end 180.323853 84.2315) (layer "Dwgs.User") (width 0.2) (fill none))
+  (gr_circle locked (center 179.362966 89.0575) (end 181.445766 89.0575) (layer "Dwgs.User") (width 0.2) (fill none))
   (gr_arc locked (start 171.656103 84.549) (mid 172.121071 83.426468) (end 173.243603 82.9615) (layer "Dwgs.User") (width 0.2))
   (gr_line locked (start 171.656103 92.8675) (end 181.874372 92.8675) (layer "Dwgs.User") (width 0.2))
   (gr_arc locked (start 170.068603 81.12) (mid 170.533571 79.997468) (end 171.656103 79.5325) (layer "Dwgs.User") (width 0.2))
   (gr_arc locked (start 183.379885 91.783576) (mid 185.329298 86.736767) (end 187.732406 81.889545) (layer "Dwgs.User") (width 0.2))
-  (gr_circle locked (center 179.362966 89.0575) (end 181.445766 89.0575) (layer "Dwgs.User") (width 0.2) (fill none))
   (gr_arc locked (start 183.379885 91.783576) (mid 182.801931 92.568329) (end 181.874372 92.8675) (layer "Dwgs.User") (width 0.2))
   (gr_arc (start 171.656103 92.8675) (mid 170.533571 92.402532) (end 170.068603 91.28) (layer "Edge.Cuts") (width 0.2))
@@
   (gr_line (start 171.656103 84.993647) (end 171.656103 84.549) (layer "Edge.Cuts") (width 0.2))
   (gr_arc (start 183.379885 91.783576) (mid 185.329298 86.736767) (end 187.732406 81.889545) (layer "Edge.Cuts") (width 0.2))
-  (gr_text "2022/09/19 PSAS ERS\nPassive Module Spring Pin Board" (at 183.2 91.3) (layer "B.SilkS")
+  (gr_text "Passive Module Spring Pin Board" (at 183.2 91.821) (layer "B.SilkS")
     (effects (font (size 0.5 0.5) (thickness 0.12)) (justify left mirror))
   )
+  (gr_text "2022/09/19" (at 171.7 91.1 270) (layer "B.SilkS")
+    (effects (font (size 0.5 0.5) (thickness 0.12)) (justify left mirror))
+  )
+  (gr_text "PSAS ERS" (at 170.6 91.1 270) (layer "B.SilkS")
+    (effects (font (size 0.5 0.5) (thickness 0.12)) (justify left mirror))
+  )
