File: controlSystem/SpringPinBoards/PassiveModule/PassiveModule.kicad_sch (KiCad schematic)
At the start: 7 parts, among them J1 Conn_01x01_Male, J2 Conn_01x01_Male, J3 Conn_01x01_Male, J4 Conn_01x01_Male, J5 Conn_01x01_Male, J6 Conn_01x01_Male, J7 Conn_02x03_Odd_Even

Commit message: Moved spring pin board libraries to psas-kicad
Parts:
- J1, J2, J3, J4, J5, J6: footprint Mill-Max-1578-3-00-15-00-00-03-0:1578-3-00-15-00-00-03-0 -> psas-footprints:Mill-Max-1578-3-00-15-00-00-03-0
- J7: footprint Wire_Pads:2x03_1.27mm_Wires_SMD -> psas-footprints:2x03_1.27mm_Wires_SMD
Changed lines of the file:
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@@
       (effects (font (size 1.27 1.27)) hide)
     )
-    (property "Footprint" "Mill-Max-1578-3-00-15-00-00-03-0:1578-3-00-15-00-00-03-0" (id 2) (at 111.76 86.36 0)
+    (property "Footprint" "psas-footprints:Mill-Max-1578-3-00-15-00-00-03-0" (id 2) (at 111.76 86.36 0)
       (effects (font (size 1.27 1.27)) hide)
     )
@@
       (effects (font (size 1.27 1.27)) hide)
     )
-    (property "Footprint" "Mill-Max-1578-3-00-15-00-00-03-0:1578-3-00-15-00-00-03-0" (id 2) (at 111.76 91.44 0)
+    (property "Footprint" "psas-footprints:Mill-Max-1578-3-00-15-00-00-03-0" (id 2) (at 111.76 91.44 0)
       (effects (font (size 1.27 1.27)) hide)
     )
@@
       (effects (font (size 1.27 1.27)) hide)
     )
-    (property "Footprint" "Mill-Max-1578-3-00-15-00-00-03-0:1578-3-00-15-00-00-03-0" (id 2) (at 111.76 81.28 0)
+    (property "Footprint" "psas-footprints:Mill-Max-1578-3-00-15-00-00-03-0" (id 2) (at 111.76 81.28 0)
       (effects (font (size 1.27 1.27)) hide)
     )
@@
       (effects (font (size 1.27 1.27)) hide)
     )
-    (property "Footprint" "Mill-Max-1578-3-00-15-00-00-03-0:1578-3-00-15-00-00-03-0" (id 2) (at 111.76 88.9 0)
+    (property "Footprint" "psas-footprints:Mill-Max-1578-3-00-15-00-00-03-0" (id 2) (at 111.76 88.9 0)
       (effects (font (size 1.27 1.27)) hide)
     )
@@
       (effects (font (size 1.27 1.27)) hide)
     )
-    (property "Footprint" "Mill-Max-1578-3-00-15-00-00-03-0:1578-3-00-15-00-00-03-0" (id 2) (at 111.76 83.82 0)
+    (property "Footprint" "psas-footprints:Mill-Max-1578-3-00-15-00-00-03-0" (id 2) (at 111.76 83.82 0)
       (effects (font (size 1.27 1.27)) hide)
     )
@@
       (effects (font (size 1.27 1.27)) hide)
     )
-    (property "Footprint" "Mill-Max-1578-3-00-15-00-00-03-0:1578-3-00-15-00-00-03-0" (id 2) (at 111.76 93.98 0)
+    (property "Footprint" "psas-footprints:Mill-Max-1578-3-00-15-00-00-03-0" (id 2) (at 111.76 93.98 0)
       (effects (font (size 1.27 1.27)) hide)
     )
@@
       (effects (font (size 1.27 1.27)) hide)
     )
-    (property "Footprint" "Wire_Pads:2x03_1.27mm_Wires_SMD" (id 2) (at 137.16 83.82 0)
+    (property "Footprint" "psas-footprints:2x03_1.27mm_Wires_SMD" (id 2) (at 137.16 83.82 0)
       (effects (font (size 1.27 1.27)) hide)
     )
@@
   (symbol_instances
     (path "/738c22c5-6909-4833-8b17-0e751fcf8a4f"
-      (reference "J1") (unit 1) (value "Conn_01x01_Male") (footprint "Mill-Max-1578-3-00-15-00-00-03-0:1578-3-00-15-00-00-03-0")
+      (reference "J1") (unit 1) (value "Conn_01x01_Male") (footprint "psas-footprints:Mill-Max-1578-3-00-15-00-00-03-0")
     )
     (path "/aa6bf315-920d-4300-b979-0b478c6668ad"
-      (reference "J2") (unit 1) (value "Conn_01x01_Male") (footprint "Mill-Max-1578-3-00-15-00-00-03-0:1578-3-00-15-00-00-03-0")
+      (reference "J2") (unit 1) (value "Conn_01x01_Male") (footprint "psas-footprints:Mill-Max-1578-3-00-15-00-00-03-0")
     )
     (path "/03114711-e2ae-408f-84db-b1cacba6a1c0"
-      (reference "J3") (unit 1) (value "Conn_01x01_Male") (footprint "Mill-Max-1578-3-00-15-00-00-03-0:1578-3-00-15-00-00-03-0")
+      (reference "J3") (unit 1) (value "Conn_01x01_Male") (footprint "psas-footprints:Mill-Max-1578-3-00-15-00-00-03-0")
     )
     (path "/82906323-e29f-4dfa-8be6-4df9935eb36b"
-      (reference "J4") (unit 1) (value "Conn_01x01_Male") (footprint "Mill-Max-1578-3-00-15-00-00-03-0:1578-3-00-15-00-00-03-0")
+      (reference "J4") (unit 1) (value "Conn_01x01_Male") (footprint "psas-footprints:Mill-Max-1578-3-00-15-00-00-03-0")
     )
     (path "/4278c2bb-de50-4758-825d-063dfd8cf611"
-      (reference "J5") (unit 1) (value "Conn_01x01_Male") (footprint "Mill-Max-1578-3-00-15-00-00-03-0:1578-3-00-15-00-00-03-0")
+      (reference "J5") (unit 1) (value "Conn_01x01_Male") (footprint "psas-footprints:Mill-Max-1578-3-00-15-00-00-03-0")
     )
     (path "/bfd23876-4cac-4374-8b2d-6ab13f099a1d"
-      (reference "J6") (unit 1) (value "Conn_01x01_Male") (footprint "Mill-Max-1578-3-00-15-00-00-03-0:1578-3-00-15-00-00-03-0")
+      (reference "J6") (unit 1) (value "Conn_01x01_Male") (footprint "psas-footprints:Mill-Max-1578-3-00-15-00-00-03-0")
     )
     (path "/c72df43e-114f-47a2-af92-4519b7c0670d"
-      (reference "J7") (unit 1) (value "Conn_02x03_Odd_Even") (footprint "Wire_Pads:2x03_1.27mm_Wires_SMD")
+      (reference "J7") (unit 1) (value "Conn_02x03_Odd_Even") (footprint "psas-footprints:2x03_1.27mm_Wires_SMD")
     )
   )
