File: controlSystem/HallSensorBoard/HallSensorBoard.kicad_sch (KiCad schematic)
At the start: 4 parts, among them J1 22-23-2031, U1 DRV5056-Q1

Commit message: Added ERS hall effect sensor board and spring pin boards
Other:
- note added: "Note: Board can be flipped 180 degrees around the vertical axis with the DRV5056 pins reversed. Place bypass cap between VCC and GND pins accordingly."
- note removed: "Note: Board is designed to be compatible with reverse pinout of the DRV5056. Place bypass cap between VCC and GND pins accordingly."
Changed lines of the file:
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@@
     (stroke (width 0) (type default) (color 0 0 0 0))
   )
-  (text "Note:\nBoard is designed to be compatible\nwith reverse pinout of the DRV5056.\nPlace bypass cap between VCC and GND pins\naccordingly."
+  (text "Note:\nBoard can be flipped 180 degrees around\nthe vertical axis with the\nDRV5056 pins reversed.\nPlace bypass cap between VCC and GND pins\naccordingly.\n"
     (at 124.46 102.87 0)
     (effects (font (size 1.27 1.27)) (justify left bottom))

Commit message: Moved hall sensor board libraries to psas-kicad
Parts:
- J1: footprint 22-23-2031:22-23-2031 -> psas-footprints:U-TI-22-23-2031
- U1: symbol DRV5056-Q1:DRV5056-Q1 -> U-TI-DRV5056-Q1-hall-effect-sensor:DRV5056-Q1
Changed lines of the file:
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@@
     (pin "2")
   )
-  (symbol (lib_id "DRV5056-Q1:DRV5056-Q1") (at 130.81 76.2 0) (unit 1)
+  (symbol (lib_id "U-TI-DRV5056-Q1-hall-effect-sensor:DRV5056-Q1") (at 130.81 76.2 0) (unit 1)
     (in_bom yes) (on_board yes) (fields_autoplaced)
     (property "Reference" "U1" (id 0) (at 130.81 66.04 0))
@@
       (effects (font (size 1.27 1.27)) (justify left))
     )
-    (property "Footprint" "22-23-2031:22-23-2031" (id 2) (at 167.64 76.2 0)
+    (property "Footprint" "psas-footprints:U-TI-22-23-2031" (id 2) (at 167.64 76.2 0)
       (effects (font (size 1.27 1.27)) hide)
     )
@@
     )
     (path "/e8f066bf-0e8c-4c32-b595-5e0eaae224e6"
-      (reference "J1") (unit 1) (value "22-23-2031") (footprint "22-23-2031:22-23-2031")
+      (reference "J1") (unit 1) (value "22-23-2031") (footprint "psas-footprints:U-TI-22-23-2031")
     )
     (path "/319d8572-9c83-470b-9ecb-02369f97b1c0"
