File: controlSystem/RecoveryBoard/kicad/RecoveryBoard/RecoveryBoard.kicad_pcb (KiCad board)
At the start: 2 copper layers, 66 x 31.8 mm, 110 parts, among them J1 From Outside World, J2 Thermistor, J3 Conn_01x04, J4 J-TE-Debug-2-1734592-0, J5 3.5mm Serial Port, J6 Sensor Board 1, J7 Sensor Board 2, J8 Conn_01x02, J9 Motor, Q1 SI7465DP-T1-E3, Q2 BSS123, U1 STM32F091C, U2 MP26123DR-LF-Z, U4 H11F1SR2M, U5 H11F1SR2M, U6 BD62120AEFJ-E2, U7 TCAN330, X1 16MHZ-2.5x2mm

Commit message: Updated recovery board with some design review things
Parts:
- added J10: 3.5mm Jack, Connector_PinHeader_2.54mm:PinHeader_1x03_P2.54mm_Vertical, F.Cu at (90.7, 100.1)
- added U3: TPS63070, psas-footprints:U-TI-TPS63070, F.Cu at (123.0, 105.4)
- moved D5 16.8 mm to (117.3, 110.0), turned to 0 degrees
- moved R14 14.8 mm to (117.3, 108.3), turned to 0 degrees
- moved C4 10.0 mm to (130.3, 105.4)
- moved C11 10.0 mm to (117.8, 105.4)
- moved C13 10.0 mm to (119.9, 105.4)
- moved C14 10.0 mm to (115.7, 105.4)
- moved C2 10.0 mm to (126.1, 105.4)
- moved C3 10.0 mm to (128.2, 105.4)
- moved R6 8.82 mm to (127.7, 102.8), turned to 180 degrees
- moved C6 3.31 mm to (121.4, 102.8), turned to 180 degrees
- moved R4 3.11 mm to (124.6, 102.8)
- moved R7 2.52 mm to (121.4, 108.0)
- moved R8 2.42 mm to (124.6, 108.0)

Commit message: Updated recovery board
Parts:
- removed U6: BD62120AEFJ-E2, Package_SO:SOIC-8-1EP_3.9x4.9mm_P1.27mm_EP2.41x3.3mm
- added D3: SS210A, Diode_SMD:D_SMA, F.Cu at (106.3, 103.3)
- added J11: Conn_01x03, Connector_Molex:Molex_KK-254_AE-6410-03A_1x03_P2.54mm_Vertical, F.Cu at (164.3, 85.2)
- added L2: 4.7uH, Inductor_SMD:L_Coilcraft_XxL4030, F.Cu at (112.2, 104.2)
- added REF**: MountingHole_2.2mm_M2, MountingHole:MountingHole_2.2mm_M2, F.Cu at (86.7, 118.2)
- added U8: BDS63150AFM-E2, psas-footprints:U-BD63150AFM, F.Cu at (149.2, 94.0)
- J1: value From Outside World -> Conn_01x06; footprint Connector_PinHeader_2.54mm:PinHeader_1x06_P2.54mm_Vertical -> Connector_Molex:Molex_KK-254_AE-6410-06A_1x06_P2.54mm_Vertical
- J10: value 3.5mm Jack -> Conn_01x02; footprint Connector_PinHeader_2.54mm:PinHeader_1x03_P2.54mm_Vertical -> Connector_Molex:Molex_KK-254_AE-6410-02A_1x02_P2.54mm_Vertical
- J2, J8, J9: footprint Connector_PinHeader_2.54mm:PinHeader_1x02_P2.54mm_Vertical -> Connector_Molex:Molex_KK-254_AE-6410-02A_1x02_P2.54mm_Vertical
- J3: footprint Connector_PinHeader_2.54mm:PinHeader_1x04_P2.54mm_Vertical -> Connector_Molex:Molex_KK-254_AE-6410-04A_1x04_P2.54mm_Vertical
- J5: value 3.5mm Serial Port -> Conn_01x03; footprint Connector_PinHeader_2.54mm:PinHeader_1x03_P2.54mm_Vertical -> Connector_Molex:Molex_KK-254_AE-6410-03A_1x03_P2.54mm_Vertical
- J6, J7: footprint Connector_PinHeader_2.54mm:PinHeader_1x03_P2.54mm_Vertical -> Connector_Molex:Molex_KK-254_AE-6410-03A_1x03_P2.54mm_Vertical
- R15: value 10k -> 33k
- U4, U5: value H11F1SR2M -> TCMT1107; footprint Package_DIP:SMDIP-6_W9.53mm_Clearance8mm -> Package_SO:SOP-4_4.4x2.6mm_P1.27mm
- moved J6 72.8 mm to (104.4, 87.4), turned to -120 degrees
- moved J9 63.4 mm to (151.3, 75.3), turned to 180 degrees
- moved J7 62.3 mm to (109.0, 79.4), turned to -120 degrees
- moved J2 61.4 mm to (115.0, 117.5)
- moved J4 60.5 mm to (171.8, 116.2), turned to 180 degrees
- moved J1 58.4 mm to (96.3, 101.2), turned to -120 degrees
- moved R22 37.2 mm to (156.6, 89.5)
- moved U5 36.1 mm to (157.2, 95.7), turned to -90 degrees
- moved R20 30.6 mm to (160.3, 89.5)
- moved J3 29.8 mm to (170.1, 95.3), turned to 120 degrees
- moved J8 29.8 mm to (173.4, 101.0), turned to 120 degrees
- moved U4 29.6 mm to (160.9, 95.7), turned to -90 degrees
- moved R23 27.8 mm to (156.3, 103.3), turned to -90 degrees
- moved REF** 23.5 mm to (183.0, 118.2)
- moved Q2 23.4 mm to (128.6, 118.2), turned to -90 degrees
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Connections:
- net UMB_ON renamed UMB_~{ON}
- J1 pad 1: /Power/ARM-OUT -> /Power/VUMB
- J1 pad 2: /Power/ARM-IN -> CANH
- J1 pad 3: /Power/VUMB -> CANH
- J1 pad 4: GND -> CANL
- J1 pad 5: T_MAIN -> CANL
- J1 pad 6: T_DROGUE -> GND
- J10 pad 1: (no net) -> /Power/ARM-IN
- J10 pad 2: (no net) -> /Power/ARM-OUT
- J5 pad 1: (no net) -> /Microcontroller/USART2_RX
- J5 pad 2: (no net) -> /Microcontroller/USART2_TX
- J5 pad 3: (no net) -> GND
- R20 pad 2: T_VLIPO -> /Microcontroller/T_DROGUE
- R22 pad 2: T_VLIPO -> /Microcontroller/T_MAIN
- U4 pad 1: T_DROGUE -> /Microcontroller/T_VLIPO
- U4 pad 3: (no net) -> /Microcontroller/ISO_DROGUE
- U4 pad 4: /Microcontroller/ISO_DROGUE -> +3.3V
- U5 pad 1: T_MAIN -> /Microcontroller/T_VLIPO
- U5 pad 3: (no net) -> /Microcontroller/ISO_MAIN
- U5 pad 4: /Microcontroller/ISO_MAIN -> +3.3V
Routing:
- net /Microcontroller/T_VLIPO: track 0.00 -> 15.1 mm
- net /Microcontroller/T_MAIN: track 0.00 -> 10.9 mm
- net /Microcontroller/T_DROGUE: track 0.00 -> 7.29 mm
- net Net-(R20-Pad1): track 0.00 -> 2.20 mm
- net Net-(R22-Pad1): track 0.00 -> 2.20 mm
Other:
- board size 66 x 31.8 mm -> 102.7 x 50.5 mm
- rule pad_to_mask_clearance: 0 -> 0.0508
- board text added: "ADD SILKSCREEN BOX FOR BOARD NUM"
- board text added: "HIGH PRESSURE MOLEX CONNS"
- board text added: "SPEC SPEAKER/ADD FOOTPRINT"
- board text added: "TODO: CHECK WHICH SIDE OF BOARD TO USE SINCE ASYMMETRICAL"
- board text added: "TODO: FIX HOLE PLACEMENTS FIX HOLES IN BOARD OUTLINE"
- board text added: "UPDATE L FOOTPRINT"

Commit message: Updated ERS board
Parts:
- added C26: 1n, Capacitor_SMD:C_0603_1608Metric, F.Cu at (163.7, 95.6)
- added C27: 100n, Capacitor_SMD:C_0603_1608Metric, F.Cu at (121.7, 91.5)
- added D4: 1N4007, Diode_SMD:D_SMA, F.Cu at (159.5, 104.2)
- added D8: D_Small, Diode_SMD:D_SMA, F.Cu at (134.3, 115.7)
- added D9: D_Small, Diode_SMD:D_SMA, F.Cu at (138.5, 115.7)
- added L1: 1.5uH, Inductor_SMD:L_Vishay_IHLP-2020, F.Cu at (135.1, 100.7)
- added LOGO1: PSAS LOGO, psas-graphics:PSAS_LOGO_10X10, F.Cu at (175.0, 121.9)
- added LS1: SMT-0440-S-R, Inductor_SMD:L_Vishay_IHLP-1616, F.Cu at (92.3, 123.3)
- added R28: Rsns, Resistor_SMD:R_1206_3216Metric, F.Cu at (124.2, 87.8)
- added R29: NP, Resistor_SMD:R_0603_1608Metric, F.Cu at (119.5, 113.6)
- added R30: NP, Resistor_SMD:R_0603_1608Metric, F.Cu at (117.7, 113.6)
- added R31: NP, Resistor_SMD:R_0603_1608Metric, F.Cu at (119.5, 116.8)
- added R32: NP, Resistor_SMD:R_0603_1608Metric, F.Cu at (117.7, 116.8)
- added R35: 60.4, Resistor_SMD:R_1206_3216Metric, F.Cu at (162.8, 92.4)
- added R36: 60.4, Resistor_SMD:R_1206_3216Metric, F.Cu at (166.0, 98.0)
- added R37: 10k, Resistor_SMD:R_0603_1608Metric, F.Cu at (116.2, 103.6)
- added R38: 10k, Resistor_SMD:R_0603_1608Metric, F.Cu at (114.3, 103.6)
- added TP32: Test-Point, psas-footprints:TP-through-hole-1X01, F.Cu at (158.5, 92.7)
- added TP33: Test-Point, psas-footprints:TP-through-hole-1X01, F.Cu at (108.8, 101.2)
- added TP34: Test-Point, psas-footprints:TP-through-hole-1X01, F.Cu at (107.0, 101.2)
- added TP35: Test-Point, psas-footprints:TP-through-hole-1X01, F.Cu at (105.2, 101.2)
- added TP36: Test-Point, psas-footprints:TP-through-hole-1X01, F.Cu at (103.4, 101.2)
- added TP37: Test-Point, psas-footprints:TP-through-hole-1X01, F.Cu at (100.2, 115.1)
- added TP38: Test-Point, psas-footprints:TP-through-hole-1X01, F.Cu at (117.9, 102.7)
- added TP39: Test-Point, psas-footprints:TP-through-hole-1X01, F.Cu at (98.4, 120.5)
- added TP40: Test-Point, psas-footprints:TP-through-hole-1X01, F.Cu at (119.7, 107.9)
- added TP41: Test-Point, psas-footprints:TP-through-hole-1X01, F.Cu at (119.7, 109.7)
- added TP42: Test-Point, psas-footprints:TP-through-hole-1X01, F.Cu at (117.9, 107.9)
- added TP43: Test-Point, psas-footprints:TP-through-hole-1X01, F.Cu at (98.4, 116.9)
- added TP44: Test-Point, psas-footprints:TP-through-hole-1X01, F.Cu at (98.4, 115.1)
- added TP45: Test-Point, psas-footprints:TP-through-hole-1X01, F.Cu at (102.0, 104.0)
- added TP46: Test-Point, psas-footprints:TP-through-hole-1X01, F.Cu at (117.9, 104.5)
- added TP47: Test-Point, psas-footprints:TP-through-hole-1X01, F.Cu at (122.0, 112.6)
- added U6: INA185, Package_TO_SOT_SMD:SOT-563, F.Cu at (123.8, 93.2)
- C11: value 22u -> 10u; footprint Capacitor_SMD:C_0805_2012Metric -> Capacitor_SMD:C_0603_1608Metric
- C4: footprint Capacitor_SMD:C_0805_2012Metric -> Capacitor_SMD:C_0603_1608Metric
- J8: value Conn_01x02 -> Conn_01x06; footprint Connector_Molex:Molex_KK-254_AE-6410-02A_1x02_P2.54mm_Vertical -> Connector_Molex:Molex_KK-254_AE-6410-06A_1x06_P2.54mm_Vertical
- L2: footprint Inductor_SMD:L_Coilcraft_XxL4030 -> Inductor_SMD:L_Vishay_IHLP-2020
- moved TP8 133.8 mm to (122.0, 114.4)
- moved TP6 133.7 mm to (126.0, 95.8)
- moved TP30 132.5 mm to (126.0, 97.6)
- moved TP31 130.0 mm to (126.0, 99.4)
- moved TP12 118.1 mm to (100.2, 107.6)
- moved TP11 117.3 mm to (102.0, 107.6)
- moved TP21 117.3 mm to (100.2, 120.5)
- moved TP20 116.4 mm to (98.4, 118.7)
- moved TP5 115.8 mm to (142.6, 115.4)
- moved TP9 110.0 mm to (140.6, 101.1)
- moved TP19 108.7 mm to (100.2, 118.7)
- moved TP15 108.3 mm to (113.0, 77.2)
- moved TP23 107.1 mm to (98.4, 122.3)
- moved TP22 106.4 mm to (100.2, 122.3)
- moved TP10 102.0 mm to (100.2, 109.4)
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Connections:
- net +12V renamed VBUS
- J4 pad 1: unconnected-(J4-Pad1) -> +5V
- J4 pad 2: unconnected-(J4-Pad1) -> +5V
- J6 pad 1: +3.3V -> /Microcontroller/HALL1
- J6 pad 2: /Microcontroller/HALL1 -> GND
- J6 pad 3: GND -> +3.3V
- J7 pad 1: +3.3V -> /Microcontroller/HALL2
- J7 pad 2: /Microcontroller/HALL2 -> GND
- J7 pad 3: GND -> +3.3V
- J8 pad 1: /Microcontroller/CANH -> /Power/VUMB
- J8 pad 2: /Microcontroller/CANL -> CANH
- Q1 pad 1: +BATT -> Net-(D8-Pad1)
- Q1 pad 2: +BATT -> Net-(D8-Pad1)
- Q1 pad 3: +BATT -> Net-(D8-Pad1)
- R26 pad 1: /Microcontroller/DEPLOY1 -> DEPLOY1
- R27 pad 1: /Microcontroller/DEPLOY2 -> DEPLOY2
- TP1 pad 1: GND -> CANH
- TP17 pad 1: /Microcontroller/SDWIO -> Net-(TP17-Pad1)
- TP18 pad 1: /Microcontroller/SWCLK -> Net-(TP18-Pad1)
- TP19 pad 1: /Microcontroller/NRST -> Net-(TP19-Pad1)
- TP2 pad 1: /Power/VUMB -> CANL
- TP26 pad 1: /Microcontroller/ISO_MAIN -> /Microcontroller/ISO_DROGUE
- TP27 pad 1: /Microcontroller/ISO_DROGUE -> /Microcontroller/ISO_MAIN
- TP3 pad 1: T_MAIN -> GND
- TP4 pad 1: T_DROGUE -> /Power/VREF33
- U1 pad 10: BATT_READ -> /Microcontroller/HALL1
- U1 pad 11: unconnected-(U1-Pad11) -> /Microcontroller/HALL2
- U1 pad 14: /Microcontroller/ISO_MAIN -> MOTOR_ILIM
- U1 pad 16: /Microcontroller/DEPLOY1 -> /Microcontroller/ISO_MAIN
- U1 pad 17: /Microcontroller/DEPLOY2 -> Net-(TP41-Pad1)
- U1 pad 18: /Microcontroller/HALL1 -> BATT_READ
- U1 pad 19: /Microcontroller/HALL2 -> MOTOR_ISENSE
- U1 pad 20: unconnected-(U1-Pad20) -> Net-(TP17-Pad1)
- U1 pad 21: unconnected-(U1-Pad21) -> /Microcontroller/AD0
- U1 pad 22: unconnected-(U1-Pad22) -> /Microcontroller/AD1
- U1 pad 25: UMB_~{ON} -> Net-(TP40-Pad1)
- U1 pad 26: unconnected-(U1-Pad26) -> Net-(TP42-Pad1)
- U1 pad 29: unconnected-(U1-Pad29) -> UMB_~{ON}
- U1 pad 38: unconnected-(U1-Pad38) -> Net-(TP43-Pad1)
- U1 pad 39: unconnected-(U1-Pad39) -> Net-(TP18-Pad1)
- U1 pad 40: unconnected-(U1-Pad40) -> DEPLOY1
- U1 pad 41: unconnected-(U1-Pad41) -> DEPLOY2
- U1 pad 42: unconnected-(U1-Pad42) -> MOTOR_~{PS}
- U1 pad 43: unconnected-(U1-Pad43) -> MOTOR_~{FAILA}
- U1 pad 45: unconnected-(U1-Pad45) -> Net-(TP19-Pad1)
- U1 pad 46: unconnected-(U1-Pad46) -> Net-(TP39-Pad1)
- U7 pad 6: /Microcontroller/CANL -> CANL
- U7 pad 7: /Microcontroller/CANH -> CANH
- U8 pad 11: /Microcontroller/DEPLOY1 -> DEPLOY1
- U8 pad 12: /Microcontroller/DEPLOY2 -> DEPLOY2
- U8 pad 20: MOTOR_VREF -> /Microcontroller/MOTOR_VREF
Routing:
- net +3.3V: track 0.00 -> 173.0 mm, vias 0 -> 17
- net /Microcontroller/USART2_TX: track 0.00 -> 120.9 mm, vias 0 -> 2
- net /Microcontroller/HALL2: track 0.00 -> 119.6 mm
- net /Microcontroller/USART2_RX: track 0.00 -> 114.7 mm, vias 0 -> 2
- net CANL: track 0.00 -> 108.1 mm, vias 0 -> 1
- net CANH: track 0.00 -> 103.5 mm, vias 0 -> 1
- net /Microcontroller/HALL1: track 0.00 -> 76.6 mm, vias 0 -> 2
- net /Power/VUMB: track 0.00 -> 74.0 mm, vias 0 -> 2
- net +5V: track 0.00 -> 64.5 mm, vias 0 -> 6
- net UMB_~{ON}: track 0.00 -> 64.2 mm, vias 0 -> 2
- net BATT_READ: track 0.00 -> 40.1 mm, vias 0 -> 2
- net Net-(J2-Pad1): track 0.00 -> 38.5 mm, vias 0 -> 4
- net MOTOR_ISENSE: track 0.00 -> 38.3 mm, vias 0 -> 3
- net MOTOR_~{PS}: track 0.00 -> 33.7 mm
- net Net-(Q1-Pad4): track 0.00 -> 32.5 mm, vias 0 -> 2
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- added copper zone on B.Cu, net +3.3V
- added copper zone on F.Cu, net +3.3V
- added copper zone on F.Cu, net +5V
- added copper zone on F.Cu, net +BATT
- added copper zone on F.Cu, net /Microcontroller/MOTOR+
- added copper zone on F.Cu, net /Microcontroller/MOTOR-
- added copper zone on F.Cu, net /Power/VUMB
- added copper zone on B.Cu, net GND
- added copper zone on F.Cu, net GND
- added copper zone on F.Cu, net Net-(C7-Pad1)
- added copper zone on F.Cu, net Net-(C8-Pad1)
- added copper zone on F.Cu, net Net-(D8-Pad1)
- added copper zone on F.Cu, net Net-(L1-Pad1)
- added copper zone on F.Cu, net Net-(L1-Pad2)
- added copper zone on F.Cu, net Net-(L2-Pad2)
- added copper zone on F.Cu, net Net-(R28-Pad1)
- added copper zone on F.Cu, net VBUS
Other:
- board size 102.7 x 50.5 mm -> 102.7 x 56.8 mm
- board text added: "2023-01-13"
- board text added: "ARM RBF"
- board text added: "BATTERY"
- board text added: "HALL SENSOR 1"
- board text added: "HALL SENSOR 2"
- board text added: "MOTOR"
- board text added: "Recovery Board v3.0"
- board text added: "SERIAL"
- board text added: "TELEMETRUM"
- board text added: "THERMISTOR"
- board text added: "UMBILICAL + CAN"
- board text removed: "ADD SILKSCREEN BOX FOR BOARD NUM"
- board text removed: "HIGH PRESSURE MOLEX CONNS"
- board text removed: "SPEC SPEAKER/ADD FOOTPRINT"
- board text removed: "TODO: CHECK WHICH SIDE OF BOARD TO USE SINCE ASYMMETRICAL"
- board text removed: "TODO: FIX HOLE PLACEMENTS FIX HOLES IN BOARD OUTLINE"
- board text removed: "UPDATE L FOOTPRINT"
