File: controlSystem/RecoveryBoard/kicad/RecoveryBoard/RecoveryBoard.kicad_sch (KiCad schematic)
At the start: 0 parts

Commit message: Updated ERS board
Parts:
- added LOGO1: PSAS LOGO, psas-graphics:PSAS_LOGO_10X10, symbol psas-graphics:PSAS LOGO
