File: controlSystem/RecoveryBoard/kicad/RecoveryBoard/RecoveryBoardMicrocontroller.kicad_sch (KiCad schematic)
At the start: 54 parts, among them J4 J-TE-Debug-2-1734592-0, J5 3.5mm Serial Port, J6 Sensor Board 1, J7 Sensor Board 2, J8 Conn_01x02, J9 Motor, Q2 BSS123, U1 STM32F091C, U4 H11F1SR2M, U5 H11F1SR2M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

Commit message: Updated recovery board with some design review things
Other:
- note added: "Add CAN address pins"
- note added: "Change to 5+A motor driver"
- note added: "Spec smaller opto-isolator"
Changed lines of the file:
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@@
+    (effects (font (size 1.27 1.27)) (justify left bottom))
+  )
+  (text "Change to 5+A motor driver" (at 340.36 88.9 0)
     (effects (font (size 1.27 1.27)) (justify left bottom))
   )
@@
     (effects (font (size 2.032 2.032)) (justify left bottom))
   )
+  (text "Spec smaller opto-isolator" (at 76.2 53.34 0)
+    (effects (font (size 1.27 1.27)) (justify left bottom))
+  )
   (text "Parachute Deployer Motor Driver" (at 307.34 73.66 0)
     (effects (font (size 2.032 2.032)) (justify left bottom))
@@
     (effects (font (size 1.27 1.27)) (justify left bottom))
   )
+  (text "Add CAN address pins" (at 170.18 167.64 0)
+    (effects (font (size 1.27 1.27)) (justify left bottom))
+  )

Commit message: Updated recovery board
Parts:
- removed J5: 3.5mm Serial Port, Connector_PinHeader_2.54mm:PinHeader_1x03_P2.54mm_Vertical, symbol Connector:AudioJack3
- removed U6: BD62120AEFJ-E2, Package_SO:SOIC-8-1EP_3.9x4.9mm_P1.27mm_EP2.41x3.3mm, symbol U-Rohm-BD62120AEFJ-E2-h-bridge-motor-driver:BD62120AEFJ-E2
- added J11, J5: Conn_01x03, Connector_Molex:Molex_KK-254_AE-6410-03A_1x03_P2.54mm_Vertical, symbol Connector_Generic:Conn_01x03
- added R28: Rsns, symbol Device:R_Small_US
- added R? (x6): NP, symbol Device:R_Small_US
- added U8: BDS63150AFM-E2, psas-footprints:U-BD63150AFM, symbol U-Rohm-BD63150AFM-E2-h-bridge-motor-driver:BDS63150AFM-E2
- J6, J7: footprint Connector_PinHeader_2.54mm:PinHeader_1x03_P2.54mm_Vertical -> Connector_Molex:Molex_KK-254_AE-6410-03A_1x03_P2.54mm_Vertical
- J8, J9: footprint Connector_PinHeader_2.54mm:PinHeader_1x02_P2.54mm_Vertical -> Connector_Molex:Molex_KK-254_AE-6410-02A_1x02_P2.54mm_Vertical
- U4, U5: value H11F1SR2M -> TCMT1107; footprint Package_DIP:SMDIP-6_W9.53mm_Clearance8mm -> Package_SO:SOP-4_4.4x2.6mm_P1.27mm; symbol U-onsemi-H11F3M-optocoupler:H11F1SR2M -> U-Vishay-TCMT1107-optocoupler:TCMT1107
Connections:
- net +12V: now also U8.24 (VCC), U8.25 (VCC), U8.26 (VCC)
- net +3.3V: now also U4.4 (IN), U5.4 (IN), R?.1, R?.1, R?.1; no longer U4.6 (IN), U5.6 (IN)
- net DEPLOY1: now also U8.11 (IN1)
- net DEPLOY2: now also U8.12 (IN2)
- net GND: now also J5.3 (Pin_3), R28.2, R?.2, R?.2, R?.2, U8.15 (TEST), U8.18 (TEST1), U8.29 (GND), U8.FIN
- net ISO_DROGUE: now also U4.3 (OUT); no longer U4.4 (OUT)
- net ISO_MAIN: now also U5.3 (OUT); no longer U5.4 (OUT)
- net MOTOR+: now also U8.1 (OUT1), U8.2 (OUT1), U8.3 (OUT1)
- net MOTOR-: now also U8.6 (OUT2), U8.7 (OUT2), U8.8 (OUT2)
- net T_DROGUE: now also R20.2, J11.2 (Pin_2); no longer U4.1 (A)
- net T_MAIN: now also R22.2, J11.3 (Pin_3); no longer U5.1 (A)
- net T_VLIPO: now also U4.1 (A), U5.1 (A), J11.1 (Pin_1); no longer R20.2, R22.2
- net USART2_RX: now also J5.1 (Pin_1)
- net USART2_TX: now also J5.2 (Pin_2)
- net UMB_~{ON}: now reaches U1.26 (PB13)
- net AD0: now reaches U1.41 (PB5)
- net AD0: now also R?.1, R?.2
- net AD1: now reaches U1.42 (PB6)
- net AD1: now also R?.1, R?.2
- net AD2: now reaches U1.43 (PB7)
- net AD2: now also R?.1, R?.2
- net UMB_ON: no longer names the net of U1.25 (PB12)
- new net: R28.1, U8.32 (RNFS), U8.33 (RNF), U8.34 (RNF), U8.35 (RNF)
- new net MOTOR_VREF: U8.20 (VREF)
- new net MOTOR_~{FAILA}: U8.16 (~{FAILA})
- new net MOTOR_~{PS}: U8.13 (~{PS})
Other:
- note added: "Adjustable vref or fixed divider from VCC?"
- note added: "Are spring pins going to cause problems with CAN bus when disconecting? What about CAN terminations?"
- note added: "Board Address"
- note added: "Connector going to 3.5 mm jack serial port"
- note added: "Deploy signals from Telemetrum flight computer"
- note added: "Drive ~{PS} low to put in sleep mode (Low power and HI-Z outputs)"
- note added: "Indicators"
- note added: "PWM Control: IN1 IN2 OUT1 OUT2 L L HI-Z HI-Z L H GND VCC H L VCC GND H H GND GND"
- note added: "TODO: More testpoints"
- note added: "TODO: VREF PIN (SEE ABOVE) SPEC SENSE RESISTOR DO WE WANT TO READ SENSE VOLTAGE? ARE WE EVEN USING CURRENT CONTROL? HOW MUCH CURRENT DOES MOTOR DRAW AT FULL DUTY RATIO"
- note added: "Telemetrum signals driven low when active, driving isolated signals high"
- note added: "VERIFY PWM AND ADC CAPABLE PINS"
- note added: "What to do with UMB_~{ON}?"
- note removed: "Add CAN address pins"
- note removed: "Change to 5+A motor driver"
- note removed: "How do the telemetrum signals work?"
- note removed: "Need diode?"
- note removed: "Spec smaller opto-isolator"
- note removed: "Use pin header for wires coming from jack?"
- note removed: "Where does CAN go to?"
- moved on the sheet: C23, C24, D7, J4, J6, J7, J9, LS1, Q2, R20, R21, R22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

Commit message: Updated ERS board
Parts:
- removed J8: Conn_01x02, Connector_Molex:Molex_KK-254_AE-6410-02A_1x02_P2.54mm_Vertical, symbol Connector_Generic:Conn_01x02
- removed R? (x2): NP, symbol Device:R_Small_US
- added C27: 100n, Capacitor_SMD:C_0603_1608Metric, symbol Device:C_Small
- added R37, R38: 10k, Resistor_SMD:R_0603_1608Metric, symbol Device:R_Small_US
- added TP33, TP34, TP35, TP36, TP37, TP38, TP39, TP40, TP41, TP42, TP43, TP44, TP45, TP46, TP47, TP8: Test-Point, psas-footprints:TP-through-hole-1X01, symbol psas-testpoint:Test-Point
- added U6: INA185, Package_TO_SOT_SMD:SOT-563, symbol psas-ics:INA185
- LS1: value Speaker -> SMT-0440-S-R; footprint (none) -> Inductor_SMD:L_Vishay_IHLP-1616; MPN (none) -> SMT-0440-S-R
- R28: footprint (none) -> Resistor_SMD:R_1206_3216Metric
- R29, R30, R31, R32: renamed from R?; footprint (none) -> Resistor_SMD:R_0603_1608Metric
Connections:
- net +3.3V: now also J6.3 (Pin_3), J7.3 (Pin_3), C27.1, U6.6 (V+); no longer J6.1 (Pin_1), J7.1 (Pin_1)
- net AD0: now also R31.2, R32.1, U1.21 (PB10); no longer U1.41 (PB5)
- net AD1: now also R29.2, R30.1, U1.22 (PB11); no longer R31.2, R32.1, U1.42 (PB6)
- net BATT_READ: now also U1.18 (PB0), TP8.1; no longer U1.10 (PA0)
- net DEPLOY1: now also U1.40 (PB4), TP33.1; no longer U1.16 (PA6)
- net DEPLOY2: now also U1.41 (PB5), TP34.1; no longer U1.17 (PA7)
- net GND: now also J6.2 (Pin_2), J7.2 (Pin_2), C27.2, R38.2, TP45.1, U6.2 (GND), U6.4 (-), U6.5 (REF); no longer J6.3 (Pin_3), J7.3 (Pin_3)
- net HALL1: now also J6.1 (Pin_1), U1.10 (PA0); no longer J6.2 (Pin_2), U1.18 (PB0)
- net HALL2: now also J7.1 (Pin_1), U1.11 (PA1); no longer J7.2 (Pin_2), U1.19 (PB1)
- net ISO_DROGUE: now also TP26.1; no longer TP27.1
- net ISO_MAIN: now also TP27.1, U1.16 (PA6); no longer TP26.1, U1.14 (PA4)
- net MOTOR_VREF: now also R37.2, R38.1, TP38.1
- net MOTOR_~{FAILA}: now also U1.43 (PB7), TP36.1
- net MOTOR_~{PS}: now also U1.42 (PB6), TP35.1
- net NRST: no longer TP19.1
- net SDWIO: no longer TP17.1
- net SWCLK: no longer TP18.1
- net UMB_~{ON}: now also U1.29 (PA8); no longer U1.26 (PB13)
- net at Q2.1 (G), R25.1, U1.28 (PB15): now also TP37.1
- net at U1.20 (PB2): now also TP17.1
- net at U1.25 (PB12): now also TP40.1
- net at U1.38 (PA15): now also TP43.1
- net at U1.39 (PB3): now also TP18.1
- net at U1.45 (PB8): now also TP19.1
- net at U1.46 (PB9): now also TP39.1
- net at R28.1, U8.32 (RNFS), U8.33 (RNF)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: now also U6.3 (+)
- net +5V: now reaches J4.1 (VBUSP), J4.2 (VBUSP)
- net +5V: now also TP44.1
- net +12V renamed VBUS
- removed net AD2: R29.2, R30.1, U1.43 (PB7)
- new net: TP42.1, U1.26 (PB13)
- new net: TP41.1, U1.17 (PA7)
- new net MOTOR_ILIM: R37.1, TP46.1, U1.14 (PA4)
- new net MOTOR_ISENSE: TP47.1, U1.19 (PB1), U6.1
- no-connect marks 5 -> 4
Other:
- note added: "Addresses: AD1 AD0 Board 0 0 Interface 0 1 Ballute 1 0 Drogue Chute 1 1 Main Chute"
- note added: "Bigger cap"
- note added: "CAP ON 5V"
- note added: "TODO: ADD NOTE SAYING OPTOISOLATOR ONLY FOR ONE BOARD? AND MOTORS/SENSORS FOR OTHERS"
- note added: "TODO: VREF PIN (SEE ABOVE) SPEC SENSE RESISTOR"
- note removed: "Adjustable vref or fixed divider from VCC?"
- note removed: "Are spring pins going to cause problems with CAN bus when disconecting? What about CAN terminations?"
- note removed: "Do we need something connected to VBUSP?"
- note removed: "Swap rx and tx?"
- note removed: "TODO: More testpoints"
- note removed: "TODO: VREF PIN (SEE ABOVE) SPEC SENSE RESISTOR DO WE WANT TO READ SENSE VOLTAGE? ARE WE EVEN USING CURRENT CONTROL? HOW MUCH CURRENT DOES MOTOR DRAW AT FULL DUTY RATIO"
- note removed: "VERIFY PWM AND ADC CAPABLE PINS"
- note removed: "What to do with UMB_~{ON}?"
- moved on the sheet: C16, C17, C18, C19, C20, C21, C22, C23, C24, D7, J11, J4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
