File: controlSystem/RecoveryBoard/kicad/RecoveryBoard/RecoveryBoardPower.kicad_sch (KiCad schematic)
At the start: 58 parts, among them J1 From Outside World, J2 Thermistor, J3 Conn_01x04, Q1 SI7465DP-T1-E3, U2 MP26123DR-LF-Z, U3 TPS63070

Commit message: Updated recovery board with some design review things
Parts:
- removed J1: From Outside World, Connector_PinHeader_2.54mm:PinHeader_1x06_P2.54mm_Vertical, symbol Connector_Generic:Conn_01x06
- removed TP1, TP2, TP3, TP4: Test-Point, psas-footprints:TP-through-hole-1X01, symbol psas-testpoint:Test-Point
- added J1: Conn_01x04, symbol Connector_Generic:Conn_01x04
- added J10: 3.5mm Jack, Connector_PinHeader_2.54mm:PinHeader_1x03_P2.54mm_Vertical, symbol Connector:AudioJack3
- U3: footprint (none) -> psas-footprints:U-TI-TPS63070
Connections:
- net ARM-IN: now also J10.T
- net ARM-OUT: now also J10.R
- net GND: now also J1.4 (Pin_4)
- net VUMB: now also J1.1 (Pin_1)
- new net CANH: J1.2 (Pin_2)
- new net CANL: J1.3 (Pin_3)
Other:
- note added: "3.5 mm jack RBF tag Shorts ARM lines to turn off power"
- note added: "CAN to other recovery boards"
- note added: "Change to 6 pin and double up CAN?"
- note added: "Todo: Fix land pattern for footprint"
- note removed: "Telemetrum Deploy Signals"
- note removed: "Tie together turn off"
- note removed: "What about T_VLIPO?"

Commit message: Updated recovery board
Parts:
- removed J10: 3.5mm Jack, Connector_PinHeader_2.54mm:PinHeader_1x03_P2.54mm_Vertical, symbol Connector:AudioJack3
- added J10: Conn_01x02, Connector_Molex:Molex_KK-254_AE-6410-02A_1x02_P2.54mm_Vertical, symbol Connector_Generic:Conn_01x02
- D3: value 1N4007 -> SS210A; footprint (none) -> Diode_SMD:D_SMA
- J1: value Conn_01x04 -> Conn_01x06; footprint (none) -> Connector_Molex:Molex_KK-254_AE-6410-06A_1x06_P2.54mm_Vertical; symbol Connector_Generic:Conn_01x04 -> Connector_Generic:Conn_01x06
- J2: footprint Connector_PinHeader_2.54mm:PinHeader_1x02_P2.54mm_Vertical -> Connector_Molex:Molex_KK-254_AE-6410-02A_1x02_P2.54mm_Vertical
- J3: footprint Connector_PinHeader_2.54mm:PinHeader_1x04_P2.54mm_Vertical -> Connector_Molex:Molex_KK-254_AE-6410-04A_1x04_P2.54mm_Vertical
- L2: footprint (none) -> Inductor_SMD:L_Coilcraft_XxL4030
- R15: value 10k -> 33k
Connections:
- net ARM-IN: now also J10.1 (Pin_1)
- net ARM-OUT: now also J10.2 (Pin_2)
- net CANH: now also J1.3 (Pin_3)
- net CANL: now also J1.4 (Pin_4), J1.5 (Pin_5); no longer J1.3 (Pin_3)
- net GND: now also J1.6 (Pin_6); no longer J1.4 (Pin_4)
- net UMB_ON renamed UMB_~{ON}
Other:
- note added: "Connector going to 3.5 mm jack RBF plug to short ARM lines Turns off power"
- note removed: "3.5 mm jack RBF tag Shorts ARM lines to turn off power"
- note removed: "Change to 6 pin and double up CAN?"

Commit message: Updated ERS board
Parts:
- removed TP8: Test-Point, psas-footprints:TP-through-hole-1X01, symbol psas-testpoint:Test-Point
- added C26: 1n, Capacitor_SMD:C_0603_1608Metric, symbol Device:C_Small
- added D8, D9: SS210A, Diode_SMD:D_SMA, symbol Device:D_Small
- added J8: Conn_01x06, Connector_Molex:Molex_KK-254_AE-6410-06A_1x06_P2.54mm_Vertical, symbol Connector_Generic:Conn_01x06
- added R35, R36: 60.4, Resistor_SMD:R_1206_3216Metric, symbol Device:R_Small_US
- added TP1, TP2, TP3, TP32, TP4: Test-Point, psas-footprints:TP-through-hole-1X01, symbol psas-testpoint:Test-Point
- C11: value 22u -> 10u; footprint Capacitor_SMD:C_0805_2012Metric -> Capacitor_SMD:C_0603_1608Metric; Field4 0805 -> 0603
- C13, C14: MPN (none) -> GRT21BR61E226ME13L
- C4: footprint Capacitor_SMD:C_0805_2012Metric -> Capacitor_SMD:C_0603_1608Metric; Field4 0805 -> 0603
- D4: footprint (none) -> Diode_SMD:D_SMA
- L1: footprint (none) -> Inductor_SMD:L_Vishay_IHLP-2020; MPN (none) -> IHLP2020CZER1R5M11
- L2: footprint Inductor_SMD:L_Coilcraft_XxL4030 -> Inductor_SMD:L_Vishay_IHLP-2020; MPN (none) -> IHLP2020BZER4R7M11
Connections:
- net +BATT: now also D9.2 (A); no longer Q1.1 (S), Q1.2 (S), Q1.3 (S)
- net CANH: now also J8.2 (Pin_2), J8.3 (Pin_3), R35.1, TP1.1
- net CANL: now also J8.4 (Pin_4), J8.5 (Pin_5), R36.2, TP2.1
- net GND: now also C26.2, J8.6 (Pin_6), TP3.1
- net VREF33: now also TP4.1
- net VUMB: now also J8.1 (Pin_1), TP32.1
- net +12V renamed VBUS
- new net: D8.1 (K), D9.1 (K), Q1.1 (S), Q1.2 (S), Q1.3 (S)
- new net: C26.1, R35.2, R36.1
- new net +5V: D8.2 (A)
Other:
- note added: "+BATT (9.0, 11.1, 12.6 V)"
- note added: "5V From debug connector"
- note added: "ADD FLIGHT READY OR SIMiLAR PLUG"
- note added: "ADD SEPARATE CONNECTOR FOR UMB INPUT ON INTERFACE BOARD?"
- note added: "Bus Power switch"
- note added: "CHANGE VALUE TO MOLEX PN"
- note added: "Connector going to 3.5 mm jack. RBF plug shorts ARM lines, turning off power."
- note added: "Doubled for redundancy"
- note added: "Remove Before Flight Plug"
- note added: "Swap for SS210A?"
- note removed: "12V Power switch"
- note removed: "Connector going to 3.5 mm jack RBF plug to short ARM lines Turns off power"
- moved on the sheet: C11, C13, C14, C2, C3, C4, C6, D5, L1, R14, R4, R6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
