File: controlSystem/RecoveryBoard/pcb/RecoveryBoardMicrocontroller.kicad_sch (KiCad schematic)
At the start: 86 parts, among them J11 0022-232031, J12 0022-232021, J4 J-TE-Debug-2-1734592-0, J5 0022-232031, J6 0022-232031, J7 0022-232031, J9 0022-232021, Q2 BSS123, Q3 PMF170XP, U1 STM32F091C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

Commit message: Made changes something something
Connections:
- net at U8.14: now also U8.28
Changed lines of the file:
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@@
+	(wire
+		(pts
+			(xy 336.55 80.01) (xy 339.09 80.01)
+		)
+		(stroke
+			(width 0)
+			(type default)
+		)
+	)
 	(wire
 		(pts
