File: controlSystem/ERSRemoteControl/ERSRemoteControl.kicad_sch (KiCad schematic)
At the start: 59 parts, among them J1 USB_C_Receptacle_USB2.0_14P, J2 B3B-XH-A, J3 0022-232031, J4 0022-232021, J5 0022-232021, J6 0022-232021, J7 0022-232021, J8 0022-232031, SW1 SW_Push, SW2 SW_Push, SW3 SW_Push, SW4 SW_Push, SW5 SW_Push, SW6 SW_Push, U1 TPS63070, U2 ESP32-S3-WROOM-1

Commit message: Final trace tweaks and checking voltages
Parts:
- R8, R9: symbol Device:R_US -> Device:R_Small_US
- renumbered C5 to C4, C4 to C5, J8 to J3, J3 to J4, J4 to J5, J5 to J6, J6 to J7, J7 to J8, R2 to R1, R1 to R2
